File: pcb/amp/riaa_pre.sch (EAGLE design)
At the start: 39 parts, among them IC1 OPA2134, IC2 OPA2134, X1 22-23-2031

Commit message: 
Parts:
- C10, C5: device amp:C-EU050-025X075 -> amp:C-EU050-045X075
Changed lines of the file:
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@@
 <?xml version="1.0" encoding="utf-8"?>
 <!DOCTYPE eagle SYSTEM "eagle.dtd">
-<eagle version="6.1">
+<eagle version="6.2">
 <drawing>
 <settings>
@@
 <part name="R7" library="amp" deviceset="R-EU_" device="0207/7" value="100k"/>
 <part name="C4" library="amp" deviceset="C-EU" device="050-025X075" value="82nF"/>
-<part name="C5" library="amp" deviceset="C-EU" device="050-025X075" value="1uF"/>
+<part name="C5" library="amp" deviceset="C-EU" device="050-045X075" value="1uF"/>
 <part name="R10" library="amp" deviceset="R-EU_" device="0207/7" value="47k"/>
 <part name="R11" library="amp" deviceset="R-EU_" device="0207/7" value="2.2k"/>
@@
 <part name="R16" library="amp" deviceset="R-EU_" device="0207/7" value="100k"/>
 <part name="C9" library="amp" deviceset="C-EU" device="050-025X075" value="82nF"/>
-<part name="C10" library="amp" deviceset="C-EU" device="050-025X075" value="1uF"/>
+<part name="C10" library="amp" deviceset="C-EU" device="050-045X075" value="1uF"/>
 <part name="AGND1" library="amp" deviceset="AGND" device=""/>
 <part name="AGND2" library="amp" deviceset="AGND" device=""/>
