File: pcb/amp_soha/amp_soha.sch (EAGLE design)
At the start: 55 parts, among them IC1 NE5535U, IC2 7812, IC3 7912, Q1 J113, Q2 J113, Q3 J113, Q4 J113

Commit message: 
Parts:
- C13, C5: device amp_soha:C-EU150-072X183 -> amp_soha:C-EU075-052X106
Changed lines of the file:
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@@
 <part name="Q2" library="amp_soha" deviceset="J113" device=""/>
 <part name="Q1" library="amp_soha" deviceset="J113" device=""/>
-<part name="C5" library="amp_soha" deviceset="C-EU" device="150-072X183" value="1uF/100V"/>
+<part name="C5" library="amp_soha" deviceset="C-EU" device="075-052X106" value="1uF/100V"/>
 <part name="P+3" library="amp_soha" deviceset="+24V" device=""/>
 <part name="IC1" library="amp_soha" deviceset="NE5535" device="U"/>
@@
 <part name="Q4" library="amp_soha" deviceset="J113" device=""/>
 <part name="Q3" library="amp_soha" deviceset="J113" device=""/>
-<part name="C13" library="amp_soha" deviceset="C-EU" device="150-072X183" value="1uF/100V"/>
+<part name="C13" library="amp_soha" deviceset="C-EU" device="075-052X106" value="1uF/100V"/>
 <part name="P+6" library="amp_soha" deviceset="+24V" device=""/>
 <part name="R14" library="amp_soha" deviceset="R-EU_" device="" value="100k"/>
