File: pcb/PR042 - tube amp (soha)/amp_soha_v2.brd (EAGLE design)
At the start: 82 x 48.9 mm, 59 parts, among them IC1 NE5535U, IC2 7812, IC3 7912, Q1 J113, Q2 J113, Q3 J113, Q4 J113

Commit message: 
Parts:
- IC1: value NE5535U -> NE5532
Changed lines of the file:
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@@
 <?xml version="1.0" encoding="utf-8"?>
 <!DOCTYPE eagle SYSTEM "eagle.dtd">
-<eagle version="6.4">
+<eagle version="6.5.0">
 <drawing>
 <settings>
@@
 <attribute name="NAME" x="28.194" y="44.831" size="1.27" layer="25" font="vector" ratio="10"/>
 </element>
-<element name="IC1" library="amp_soha" package="SO08" value="NE5535U" x="45.085" y="25.4" smashed="yes" rot="MR180">
+<element name="IC1" library="amp_soha" package="SO08" value="NE5532" x="45.085" y="25.4" smashed="yes" rot="MR180">
 <attribute name="NAME" x="41.0845" y="24.13" size="1.27" layer="26" font="vector" ratio="10" rot="MR90"/>
 </element>
