File: pcb/PR042 - tube amp (soha)/amp_soha_v3.brd (EAGLE design)
At the start: 82 x 48.9 mm, 59 parts, among them IC1 NE5532, IC2 7812, IC3 7912, Q1 J113, Q2 J113, Q3 J113, Q4 J113

Commit message: 
Parts:
- moved IC4 2.54 mm to (57.8, 7.94)
- moved R11 2.54 mm to (60.3, 6.35)
- moved R9 2.54 mm to (55.2, 6.35)
Routing:
- net N$6: track 140.7 -> 138.2 mm
- net N$3: track 44.5 -> 42.0 mm
Changed lines of the file:
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@@
 <?xml version="1.0" encoding="utf-8"?>
 <!DOCTYPE eagle SYSTEM "eagle.dtd">
-<eagle version="6.5.0">
+<eagle version="6.4">
 <drawing>
 <settings>
@@
 <attribute name="NAME" x="77.089" y="10.9982" size="1.27" layer="25" font="vector" ratio="10"/>
 </element>
-<element name="R9" library="amp_soha" package="R0805" value="1k3" x="55.245" y="3.81" smashed="yes" rot="MR0">
-<attribute name="NAME" x="56.1975" y="4.7625" size="1.27" layer="26" font="vector" ratio="10" rot="MR0"/>
-</element>
-<element name="R11" library="amp_soha" package="R0805" value="11k" x="60.325" y="3.81" smashed="yes" rot="MR0">
-<attribute name="NAME" x="61.9125" y="4.7625" size="1.27" layer="26" font="vector" ratio="10" rot="MR0"/>
+<element name="R9" library="amp_soha" package="R0805" value="1k3" x="55.245" y="6.35" smashed="yes" rot="MR0">
+<attribute name="NAME" x="56.1975" y="7.3025" size="1.27" layer="26" font="vector" ratio="10" rot="MR0"/>
+</element>
+<element name="R11" library="amp_soha" package="R0805" value="11k" x="60.325" y="6.35" smashed="yes" rot="MR0">
+<attribute name="NAME" x="61.9125" y="7.3025" size="1.27" layer="26" font="vector" ratio="10" rot="MR0"/>
 </element>
 <element name="C12" library="amp_soha" package="E2,5-6" value="47uF/16V" x="45.4025" y="7.9375" smashed="yes" rot="R270">
@@
 <attribute name="VALUE" x="49.53" y="24.13" size="1.27" layer="27" rot="R270"/>
 </element>
-<element name="IC4" library="amp_soha" package="337TS" value="" x="57.785" y="5.3975" smashed="yes" rot="R180">
-<attribute name="NAME" x="56.515" y="3.6068" size="1.27" layer="25" font="vector" ratio="10"/>
-<attribute name="VALUE" x="62.865" y="13.0175" size="1.27" layer="27" ratio="10" rot="R180"/>
+<element name="IC4" library="amp_soha" package="337TS" value="" x="57.785" y="7.9375" smashed="yes" rot="R180">
+<attribute name="NAME" x="56.515" y="6.1468" size="1.27" layer="25" font="vector" ratio="10"/>
+<attribute name="VALUE" x="62.865" y="15.5575" size="1.27" layer="27" ratio="10" rot="R180"/>
 </element>
 <element name="TRIM_R" library="amp_soha" package="RTRIM3296W" value="2k" x="12.7" y="9.8425" smashed="yes" rot="R180">
@@
 <wire x1="72.39" y1="10.16" x2="72.39" y2="12.7" width="0.4064" layer="16"/>
 <wire x1="72.39" y1="12.7" x2="71.12" y2="13.97" width="0.4064" layer="16"/>
-<wire x1="57.785" y1="7.9375" x2="57.785" y2="12.7" width="0.4064" layer="16"/>
+<wire x1="57.785" y1="10.4775" x2="57.785" y2="12.7" width="0.4064" layer="16"/>
 <wire x1="57.785" y1="12.7" x2="59.055" y2="13.97" width="0.4064" layer="16"/>
 <wire x1="59.055" y1="13.97" x2="66.04" y2="13.97" width="0.4064" layer="16"/>
@@
 <contactref element="R9" pad="1"/>
 <contactref element="IC4" pad="1"/>
-<wire x1="56.195" y1="3.81" x2="59.375" y2="3.81" width="0.4064" layer="16"/>
-<wire x1="60.325" y1="7.9375" x2="60.325" y2="5.3975" width="0.4064" layer="16"/>
-<wire x1="60.325" y1="5.3975" x2="59.3725" y2="4.445" width="0.4064" layer="16"/>
-<wire x1="59.3725" y1="4.445" x2="59.3725" y2="3.8125" width="0.4064" layer="16"/>
-<wire x1="59.3725" y1="3.8125" x2="59.375" y2="3.81" width="0.4064" layer="16"/>
+<wire x1="56.195" y1="6.35" x2="59.375" y2="6.35" width="0.4064" layer="16"/>
+<wire x1="60.325" y1="10.4775" x2="60.325" y2="7.9375" width="0.4064" layer="16"/>
+<wire x1="60.325" y1="7.9375" x2="59.3725" y2="6.985" width="0.4064" layer="16"/>
+<wire x1="59.3725" y1="6.985" x2="59.3725" y2="6.3525" width="0.4064" layer="16"/>
+<wire x1="59.3725" y1="6.3525" x2="59.375" y2="6.35" width="0.4064" layer="16"/>
 </signal>
 <signal name="-12.6V">
@@
 <wire x1="37.25" y1="20.142" x2="31.992" y2="25.4" width="0.4064" layer="16"/>
 <wire x1="31.992" y1="25.4" x2="31.75" y2="25.4" width="0.4064" layer="16"/>
-<wire x1="31.75" y1="3.81" x2="45.4025" y2="3.81" width="0.4064" layer="16"/>
-<wire x1="45.4025" y1="3.81" x2="54.295" y2="3.81" width="0.4064" layer="16"/>
-<wire x1="45.4025" y1="6.6675" x2="45.4025" y2="3.81" width="0.4064" layer="16"/>
-<wire x1="55.245" y1="7.9375" x2="54.61" y2="7.3025" width="0.4064" layer="16"/>
-<wire x1="54.61" y1="7.3025" x2="54.61" y2="4.13" width="0.4064" layer="16"/>
+<wire x1="55.245" y1="10.4775" x2="54.61" y2="9.8425" width="0.4064" layer="16"/>
+<wire x1="54.61" y1="9.8425" x2="54.61" y2="6.67" width="0.4064" layer="16"/>
 <wire x1="31.75" y1="3.81" x2="30.48" y2="5.08" width="0.4064" layer="16"/>
 <wire x1="30.48" y1="5.08" x2="30.48" y2="11.43" width="0.4064" layer="16"/>
@@
 <wire x1="37.25" y1="14.0725" x2="35.8775" y2="12.7" width="0.4064" layer="16"/>
 <wire x1="35.8775" y1="12.7" x2="31.75" y2="12.7" width="0.4064" layer="16"/>
-<wire x1="54.61" y1="4.13" x2="54.295" y2="3.81" width="0.4064" layer="16"/>
+<wire x1="54.61" y1="6.67" x2="54.295" y2="6.35" width="0.4064" layer="16"/>
+<wire x1="54.295" y1="6.35" x2="45.72" y2="6.35" width="0.4064" layer="16"/>
+<wire x1="45.72" y1="6.35" x2="45.4025" y2="6.35" width="0.4064" layer="16"/>
+<wire x1="45.4025" y1="6.35" x2="45.4025" y2="6.6675" width="0.4064" layer="16"/>
+<wire x1="45.4025" y1="6.6675" x2="45.72" y2="6.35" width="0.4064" layer="16"/>
+<wire x1="45.72" y1="6.35" x2="45.72" y2="5.08" width="0.4064" layer="16"/>
+<wire x1="45.72" y1="5.08" x2="44.45" y2="3.81" width="0.4064" layer="16"/>
+<wire x1="44.45" y1="3.81" x2="31.75" y2="3.81" width="0.4064" layer="16"/>
 </signal>
 <signal name="N$7">
@@
 <wire x1="59.69" y1="48.26" x2="58.42" y2="46.99" width="0.4064" layer="16"/>
 <wire x1="58.42" y1="46.99" x2="58.42" y2="43.19" width="0.4064" layer="16"/>
-<wire x1="57.15" y1="5.3975" x2="56.515" y2="6.0325" width="0.4064" layer="16"/>
-<wire x1="56.515" y1="6.0325" x2="56.515" y2="16.51" width="0.4064" layer="16"/>
-<wire x1="57.15" y1="5.3975" x2="58.42" y2="5.3975" width="0.4064" layer="16"/>
-<wire x1="58.42" y1="5.3975" x2="59.055" y2="6.0325" width="0.4064" layer="16"/>
-<wire x1="59.055" y1="6.0325" x2="59.055" y2="10.795" width="0.4064" layer="16"/>
-<wire x1="59.055" y1="10.795" x2="59.69" y2="11.43" width="0.4064" layer="16"/>
-<wire x1="59.69" y1="11.43" x2="67.31" y2="11.43" width="0.4064" layer="16"/>
-<wire x1="67.31" y1="11.43" x2="68.58" y2="10.16" width="0.4064" layer="16"/>
-<wire x1="68.58" y1="10.16" x2="68.58" y2="8.89" width="0.4064" layer="16"/>
+<wire x1="57.15" y1="7.9375" x2="56.515" y2="8.5725" width="0.4064" layer="16"/>
+<wire x1="56.515" y1="8.5725" x2="56.515" y2="16.51" width="0.4064" layer="16"/>
+<wire x1="57.15" y1="7.9375" x2="58.42" y2="7.9375" width="0.4064" layer="16"/>
+<wire x1="58.42" y1="7.9375" x2="59.055" y2="8.5725" width="0.4064" layer="16"/>
+<wire x1="59.055" y1="8.5725" x2="59.055" y2="12.065" width="0.4064" layer="16"/>
+<wire x1="59.055" y1="12.065" x2="59.69" y2="12.7" width="0.4064" layer="16"/>
+<wire x1="59.69" y1="12.7" x2="67.31" y2="12.7" width="0.4064" layer="16"/>
+<wire x1="67.31" y1="12.7" x2="68.58" y2="11.43" width="0.4064" layer="16"/>
+<wire x1="68.58" y1="11.43" x2="68.58" y2="8.89" width="0.4064" layer="16"/>
 <wire x1="68.58" y1="8.89" x2="69.85" y2="7.62" width="0.4064" layer="16"/>
 <wire x1="74.93" y1="7.62" x2="76.2" y2="8.89" width="0.4064" layer="16"/>
