File: pcb/PR043 - pedal fuzz factory/fuzz.brd (EAGLE design)
At the start: 67.9 x 19.7 mm, 25 parts, among them T1 AC128, T2 AC128, T3 2N3904

Commit message: 
Parts:
- R6: value 5k1 -> 5k6
Changed lines of the file:
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@@
 <?xml version="1.0" encoding="utf-8"?>
 <!DOCTYPE eagle SYSTEM "eagle.dtd">
-<eagle version="6.4">
+<eagle version="6.5.0">
 <drawing>
 <settings>
@@
 <attribute name="NAME" x="17.907" y="12.954" size="1.27" layer="25" font="vector" ratio="10"/>
 </element>
-<element name="R6" library="fuzz" package="0207/7" value="5k1" x="55.88" y="7.62" smashed="yes" rot="R270">
+<element name="R6" library="fuzz" package="0207/7" value="5k6" x="55.88" y="7.62" smashed="yes" rot="R270">
 <attribute name="NAME" x="56.388" y="0.635" size="1.27" layer="25" font="vector" ratio="10" rot="R90"/>
 </element>
