File: pcb/PR043 - pedal fuzz factory/fuzz.sch (EAGLE design)
At the start: 25 parts, among them T1 AC128, T2 AC128, T3 2N3904

Commit message: 
Parts:
- R6: value 5k1 -> 5k6
Changed lines of the file:
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@@
 <?xml version="1.0" encoding="utf-8"?>
 <!DOCTYPE eagle SYSTEM "eagle.dtd">
-<eagle version="6.4">
+<eagle version="6.5.0">
 <drawing>
 <settings>
@@
 <setting verticaltext="up"/>
 </settings>
-<grid distance="0.1" unitdist="inch" unit="inch" style="lines" multiple="1" display="no" altdistance="0.05" altunitdist="inch" altunit="inch"/>
+<grid distance="0.1" unitdist="inch" unit="inch" style="lines" multiple="1" display="no" altdistance="0.01" altunitdist="inch" altunit="inch"/>
 <layers>
 <layer number="1" name="Top" color="4" fill="1" visible="no" active="no"/>
@@
 <part name="DRIVE" library="fuzz" deviceset="POTENTIOMETER_" device="" value="10kB"/>
 <part name="C2" library="fuzz" deviceset="CPOL-EU" device="E2.5-6" value="10uF"/>
-<part name="R6" library="fuzz" deviceset="R-EU_" device="0207/7" value="5k1"/>
+<part name="R6" library="fuzz" deviceset="R-EU_" device="0207/7" value="5k6"/>
 <part name="VOL" library="fuzz" deviceset="POTENTIOMETER_" device="" value="5kB"/>
 <part name="C5" library="fuzz" deviceset="CPOL-EU" device="E2.5-6" value="10uF"/>
