File: pcb/PR044 - king of tone (pedal)/kingoftone_v1.brd (EAGLE design)
At the start: 74.8 x 49.6 mm, 84 parts, among them IC1 NE5535P, IC2 NE5535P

Commit message: 
Parts:
- D1, D14: value 1N4004C -> 1N5817
- D10, D11, D2, D3, D5, D6, D8, D9: value 1N4004C -> MA856 (1N4148)
- D12, D13, D4, D7: value 1N4004C -> 1S1588 (1N4001)
Changed lines of the file:
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@@
 <element name="C4" library="kingoftone" package="C050-025X075" value="100nF" x="11.43" y="29.21" rot="R90"/>
 <element name="R10" library="kingoftone" package="0207/5V" value="220k" x="20.32" y="21.59" rot="R180"/>
-<element name="D2" library="kingoftone" package="DO41-5" value="1N4004C" x="12.7" y="19.05"/>
-<element name="D3" library="kingoftone" package="DO41-5" value="1N4004C" x="20.32" y="19.05"/>
+<element name="D2" library="kingoftone" package="DO41-5" value="MA856 (1N4148)" x="12.7" y="19.05"/>
+<element name="D3" library="kingoftone" package="DO41-5" value="MA856 (1N4148)" x="20.32" y="19.05"/>
 <element name="R12" library="kingoftone" package="0207/5V" value="6k8" x="12.7" y="21.59"/>
-<element name="D5" library="kingoftone" package="DO41-5" value="1N4004C" x="12.7" y="16.51" rot="R180"/>
-<element name="D6" library="kingoftone" package="DO41-5" value="1N4004C" x="20.32" y="16.51" rot="R180"/>
+<element name="D5" library="kingoftone" package="DO41-5" value="MA856 (1N4148)" x="12.7" y="16.51" rot="R180"/>
+<element name="D6" library="kingoftone" package="DO41-5" value="MA856 (1N4148)" x="20.32" y="16.51" rot="R180"/>
 <element name="SW1" library="kingoftone" package="EDG-02" value="" x="26.67" y="29.21"/>
 <element name="R5" library="kingoftone" package="0207/5V" value="1k" x="27.94" y="21.59" rot="R180"/>
-<element name="D4" library="kingoftone" package="DO41-5" value="1N4004C" x="27.94" y="19.05"/>
-<element name="D7" library="kingoftone" package="DO41-5" value="1N4004C" x="27.94" y="16.51" rot="R180"/>
+<element name="D4" library="kingoftone" package="DO41-5" value="1S1588 (1N4001)" x="27.94" y="19.05"/>
+<element name="D7" library="kingoftone" package="DO41-5" value="1S1588 (1N4001)" x="27.94" y="16.51" rot="R180"/>
 <element name="TONE.1" library="kingoftone" package="1X03" value="25kB" x="3.81" y="25.4" rot="R90"/>
 <element name="R6" library="kingoftone" package="0207/5V" value="6k8" x="12.7" y="13.97"/>
@@
 <element name="OUT.1" library="kingoftone" package="1X02" value="" x="11.43" y="4.445" rot="R180"/>
 <element name="PWR.1" library="kingoftone" package="1X02" value="" x="26.67" y="46.355"/>
-<element name="D1" library="kingoftone" package="DO41-5" value="1N4004C" x="31.115" y="41.91"/>
+<element name="D1" library="kingoftone" package="DO41-5" value="1N5817" x="31.115" y="41.91"/>
 <element name="C6" library="kingoftone" package="E2,5-6" value="100uF" x="33.02" y="32.0675"/>
 <element name="R3" library="kingoftone" package="0207/5V" value="47k" x="31.115" y="39.37" rot="R180"/>
@@
 <element name="C15" library="kingoftone" package="C050-025X075" value="100nF" x="48.26" y="29.21" rot="R90"/>
 <element name="R21" library="kingoftone" package="0207/5V" value="220k" x="57.15" y="21.59" rot="R180"/>
-<element name="D8" library="kingoftone" package="DO41-5" value="1N4004C" x="49.53" y="19.05"/>
-<element name="D9" library="kingoftone" package="DO41-5" value="1N4004C" x="57.15" y="19.05"/>
+<element name="D8" library="kingoftone" package="DO41-5" value="MA856 (1N4148)" x="49.53" y="19.05"/>
+<element name="D9" library="kingoftone" package="DO41-5" value="MA856 (1N4148)" x="57.15" y="19.05"/>
 <element name="R22" library="kingoftone" package="0207/5V" value="6k8" x="49.53" y="21.59"/>
-<element name="D10" library="kingoftone" package="DO41-5" value="1N4004C" x="49.53" y="16.51" rot="R180"/>
-<element name="D11" library="kingoftone" package="DO41-5" value="1N4004C" x="57.15" y="16.51" rot="R180"/>
+<element name="D10" library="kingoftone" package="DO41-5" value="MA856 (1N4148)" x="49.53" y="16.51" rot="R180"/>
+<element name="D11" library="kingoftone" package="DO41-5" value="MA856 (1N4148)" x="57.15" y="16.51" rot="R180"/>
 <element name="SW2" library="kingoftone" package="EDG-02" value="" x="63.5" y="29.21"/>
 <element name="R23" library="kingoftone" package="0207/5V" value="1k" x="64.77" y="21.59" rot="R180"/>
-<element name="D12" library="kingoftone" package="DO41-5" value="1N4004C" x="64.77" y="19.05"/>
-<element name="D13" library="kingoftone" package="DO41-5" value="1N4004C" x="64.77" y="16.51" rot="R180"/>
+<element name="D12" library="kingoftone" package="DO41-5" value="1S1588 (1N4001)" x="64.77" y="19.05"/>
+<element name="D13" library="kingoftone" package="DO41-5" value="1S1588 (1N4001)" x="64.77" y="16.51" rot="R180"/>
 <element name="TONE.2" library="kingoftone" package="1X03" value="25kB" x="40.64" y="25.4" rot="R90"/>
 <element name="R24" library="kingoftone" package="0207/5V" value="6k8" x="49.53" y="13.97"/>
@@
 <element name="OUT.2" library="kingoftone" package="1X02" value="" x="48.26" y="4.445" rot="R180"/>
 <element name="PWR.2" library="kingoftone" package="1X02" value="" x="63.5" y="46.355"/>
-<element name="D14" library="kingoftone" package="DO41-5" value="1N4004C" x="67.945" y="41.91"/>
+<element name="D14" library="kingoftone" package="DO41-5" value="1N5817" x="67.945" y="41.91"/>
 <element name="C19" library="kingoftone" package="E2,5-6" value="100uF" x="69.85" y="32.0675"/>
 <element name="R26" library="kingoftone" package="0207/5V" value="47k" x="67.945" y="39.37" rot="R180"/>
