File: pcb/PR044 - king of tone (pedal)/kingoftone_v2.sch (EAGLE design)
At the start: 84 parts, among them IC1 NE5535P, IC2 NE5535P

Commit message: 
Parts:
- removed C11, C13, C14, C16, C17: 10nF, kingoftone:C-EU050-025X075
- removed C12: 100pF, kingoftone:C-EU050-025X075
- removed C15: 100nF, kingoftone:C-EU050-025X075
- removed C18: 1uF, kingoftone:C-EU050-025X075
- removed C19, C20: 100uF, kingoftone:CPOL-EUE2.5-6
- removed D10, D11, D8, D9: MA856 (1N4148), kingoftone:1N4004C
- removed D12, D13: 1S1588 (1N4001), kingoftone:1N4004C
- removed D14: 1N5817, kingoftone:1N4004C
- removed GAIN.2: 100kB, kingoftone:POTENTIOMETER_
- removed IC2: NE5535P, kingoftone:NE5535P
- removed IN.2, LED.2, OUT.2, PWR.2: (no value), kingoftone:PINHD-1X2
- removed LED2: (no value), kingoftone:LED3MM
- removed PRES.2: 50k, kingoftone:POTENTIOMETER_CT6
- removed R15, R16, R25: 1M, kingoftone:R-EU_0207/5V
- removed R17: 27k, kingoftone:R-EU_0207/5V
- removed R18: 33k, kingoftone:R-EU_0207/5V
- removed R19, R20: 10k, kingoftone:R-EU_0207/5V
- removed R21: 220k, kingoftone:R-EU_0207/5V
- removed R22, R24: 6k8, kingoftone:R-EU_0207/5V
- removed R23, R28: 1k, kingoftone:R-EU_0207/5V
- removed R26, R27: 47k, kingoftone:R-EU_0207/5V
- removed SW1, SW2: (no value), kingoftone:SW_DIP-2
- removed TONE.2: 25kB, kingoftone:POTENTIOMETER_
- removed VOL.2: 100kA, kingoftone:POTENTIOMETER_
- added S1: SWS002, kingoftone:SWS002
- C1, C10, C2, C3, C4, C5, C8, C9: device kingoftone:C-EU050-025X075 -> kingoftone:C-EUC0805K
- C6, C7: device kingoftone:CPOL-EUE2.5-6 -> kingoftone:CPOL-EUD
- D1: value 1N5817 -> ES1; device kingoftone:1N4004C -> kingoftone:ES1
- D2, D3, D5, D6: value MA856 (1N4148) -> 1N4148; device kingoftone:1N4004C -> kingoftone:1N4148
- D4, D7: value 1S1588 (1N4001) -> S1M; device kingoftone:1N4004C -> kingoftone:S1M
- IC1: value NE5535P -> NE5535U; device kingoftone:NE5535P -> kingoftone:NE5535U
- R1, R10, R11, R12, R13, R14, R2, R3, R4, R5, R6, R7, R8, R9: device kingoftone:R-EU_0207/5V -> kingoftone:R-EU_0805
Connections:
- removed net N$27: C11.1, IN.2.2, R15.2
- removed net N$28: C11.2, IC2A.+IN, R16.1
- removed net N$29: C12.1, IC2A.-IN, R17.2, R18.2, R19.1
- removed net N$30: C12.2, GAIN.2.3, IC2A.OUT
- removed net N$31: C13.1, R17.1
- removed net N$32: C14.2, R18.1
- removed net N$33: GAIN.2.1, R19.2
- removed net N$34: C15.1, R20.1
- removed net N$35: GAIN.2.2, R20.2
- removed net N$36: C15.2, IC2B.-IN, R21.2, R22.2
- removed net N$37: IC2B.OUT, R21.1, R23.2, SW2.4
- removed net N$38: D8.A, D9.C
- removed net N$39: D10.A, D8.C, R22.1
- removed net N$40: D10.C, D11.A
- removed net N$41: D11.C, D9.A, SW2.1
- removed net N$42: D12.A, D13.C, SW2.2
- removed net N$43: R24.1, TONE.2.3
- removed net N$44: C16.1, TONE.2.1
- removed net N$45: C17.2, PRES.2.2
- removed net N$46: PRES.2.1, PRES.2.3, R24.2, VOL.2.2
- removed net N$47: D12.C, D13.A, R23.1, TONE.2.2
- removed net N$48: C18.1, VOL.2.3
- removed net N$49: C18.2, OUT.2.2, R25.2
- removed net N$50: D14.A, PWR.2.2
- removed net N$51: LED2.A, R28.1
- removed net N$52: LED.2.2, LED2.C
- net +4.5V: now also S1.3; no longer C16.2, C17.1, C20.+, IC2B.+IN, R16.2, R26.1, R27.2, SW1.3, SW2.3, VOL.2.1
- net +9V: no longer C19.+, D14.C, IC2A.V+, R26.2, R28.2
- net GND: no longer C13.2, C14.1, C19.-, C20.-, IC2A.V-, IN.2.1, LED.2.1, OUT.2.1, PWR.2.1, R15.1, R25.1, R27.1
- net N$11: now also S1.4; no longer SW1.4
- net N$15: now also S1.1; no longer SW1.1
- net N$17: now also S1.2; no longer SW1.2
