File: pcb/PR035 - soha (tube amp)/amp_soha_v4.brd (EAGLE design)
At the start: 81.1 x 45.8 mm, 57 parts, among them IC1 NE5532, IC2 7812, IC3 7912, Q1 J113, Q2 J113, Q3 J113, Q4 J113

Commit message: 
Parts:
- C10, C12, C7: value 47uF/16V -> 100uF/16V
- C11: value 47uF/35V -> 100uF/35V
Changed lines of the file:
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@@
 <?xml version="1.0" encoding="utf-8"?>
 <!DOCTYPE eagle SYSTEM "eagle.dtd">
-<eagle version="6.4">
+<eagle version="6.5.0">
 <drawing>
 <settings>
@@
 <attribute name="NAME" x="75.8825" y="30.1625" size="1.27" layer="26" font="vector" ratio="10" rot="MR0"/>
 </element>
-<element name="C11" library="amp_soha" package="E2,5-6" value="47uF/35V" x="60.325" y="22.86" smashed="yes">
+<element name="C11" library="amp_soha" package="E2,5-6" value="100uF/35V" x="60.325" y="22.86" smashed="yes">
 <attribute name="NAME" x="58.674" y="18.6182" size="1.27" layer="25" font="vector" ratio="10"/>
 </element>
@@
 <attribute name="NAME" x="44.45" y="22.225" size="1.27" layer="26" font="vector" ratio="10" rot="MR270"/>
 </element>
-<element name="C12" library="amp_soha" package="E2,5-6" value="47uF/16V" x="54.61" y="22.86" smashed="yes" rot="R180">
+<element name="C12" library="amp_soha" package="E2,5-6" value="100uF/16V" x="54.61" y="22.86" smashed="yes" rot="R180">
 <attribute name="NAME" x="52.832" y="18.669" size="1.27" layer="25" font="vector" ratio="10"/>
 </element>
@@
 <attribute name="NAME" x="56.3118" y="32.004" size="1.27" layer="25" font="vector" ratio="10" rot="R90"/>
 </element>
-<element name="C10" library="amp_soha" package="E2,5-6" value="47uF/16V" x="59.055" y="41.275" smashed="yes" rot="R180">
+<element name="C10" library="amp_soha" package="E2,5-6" value="100uF/16V" x="59.055" y="41.275" smashed="yes" rot="R180">
 <attribute name="NAME" x="57.277" y="38.989" size="1.27" layer="25" font="vector" ratio="10"/>
 </element>
-<element name="C7" library="amp_soha" package="E2,5-6" value="47uF/16V" x="59.055" y="4.445" smashed="yes">
+<element name="C7" library="amp_soha" package="E2,5-6" value="100uF/16V" x="59.055" y="4.445" smashed="yes">
 <attribute name="NAME" x="58.2295" y="2.159" size="1.27" layer="25" font="vector" ratio="10"/>
 </element>
