File: pcb/PR037 - king of tone (pedal)/kingoftone_v1.brd (EAGLE design)
At the start: 74.8 x 49.6 mm, 84 parts, among them IC1 NE5535P, IC2 NE5535P

Commit message: 
Routing:
- net +4.5V: track 75.1 -> 78.1 mm
Changed lines of the file:
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@@
 <setting verticaltext="up"/>
 </settings>
-<grid distance="0.05" unitdist="inch" unit="mm" style="lines" multiple="1" display="yes" altdistance="0.0125" altunitdist="inch" altunit="inch"/>
+<grid distance="0.05" unitdist="inch" unit="inch" style="lines" multiple="1" display="yes" altdistance="0.0125" altunitdist="inch" altunit="inch"/>
 <layers>
 <layer number="1" name="Top" color="4" fill="1" visible="yes" active="yes"/>
@@
 <wire x1="66.675" y1="44.1325" x2="63.5" y2="44.1325" width="0.4064" layer="16"/>
 <wire x1="63.5" y1="44.1325" x2="63.5" y2="48.5775" width="0.4064" layer="16"/>
-<polygon width="0.4064" layer="16" isolate="0.4064">
+<polygon width="0.4064" layer="16" isolate="0.3048">
 <vertex x="38.1" y="-1.27"/>
 <vertex x="38.1" y="52.07"/>
@@
 <vertex x="76.2" y="-1.27"/>
 </polygon>
-<wire x1="60.96" y1="39.37" x2="64.135" y2="37.465" width="0" layer="19" extent="16-16"/>
+<wire x1="64.135" y1="37.465" x2="63.1825" y2="38.4175" width="0.4064" layer="16"/>
+<wire x1="63.1825" y1="38.4175" x2="62.865" y2="38.4175" width="0.4064" layer="16"/>
+<wire x1="62.865" y1="38.4175" x2="61.9125" y2="39.37" width="0.4064" layer="16"/>
 <wire x1="34.29" y1="26.3525" x2="40.64" y2="12.7" width="0" layer="19" extent="1-1"/>
 </signal>
