File: pcb/PR025 - amp/radio_v2.brd (EAGLE design)
At the start: 30.5 x 44.5 mm, 15 parts, among them IC1 LM1117S, U1 TEA5767

Commit message: 
Parts:
- added U$5: (no value), amp:FOX-1
Routing:
- net +3V3: vias 1 -> 4
Other:
- board text added: "RADIO"
Changed lines of the file:
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@@
 <layer number="25" name="tNames" color="7" fill="1" visible="yes" active="yes"/>
 <layer number="26" name="bNames" color="7" fill="1" visible="yes" active="yes"/>
-<layer number="27" name="tValues" color="7" fill="1" visible="no" active="yes"/>
-<layer number="28" name="bValues" color="7" fill="1" visible="no" active="yes"/>
+<layer number="27" name="tValues" color="7" fill="1" visible="yes" active="yes"/>
+<layer number="28" name="bValues" color="7" fill="1" visible="yes" active="yes"/>
 <layer number="29" name="tStop" color="7" fill="3" visible="no" active="yes"/>
 <layer number="30" name="bStop" color="7" fill="6" visible="no" active="yes"/>
@@
 <layer number="39" name="tKeepout" color="4" fill="11" visible="yes" active="yes"/>
 <layer number="40" name="bKeepout" color="1" fill="11" visible="yes" active="yes"/>
-<layer number="41" name="tRestrict" color="4" fill="10" visible="no" active="yes"/>
-<layer number="42" name="bRestrict" color="1" fill="10" visible="no" active="yes"/>
-<layer number="43" name="vRestrict" color="2" fill="10" visible="no" active="yes"/>
+<layer number="41" name="tRestrict" color="4" fill="10" visible="yes" active="yes"/>
+<layer number="42" name="bRestrict" color="1" fill="10" visible="yes" active="yes"/>
+<layer number="43" name="vRestrict" color="2" fill="10" visible="yes" active="yes"/>
 <layer number="44" name="Drills" color="7" fill="1" visible="no" active="yes"/>
 <layer number="45" name="Holes" color="7" fill="1" visible="yes" active="yes"/>
@@
 <wire x1="30.48" y1="44.45" x2="30.48" y2="0" width="0.4064" layer="20"/>
 <wire x1="30.48" y1="0" x2="0" y2="0" width="0.4064" layer="20"/>
-<wire x1="30.48" y1="22.225" x2="0" y2="22.225" width="0.4064" layer="49"/>
-<wire x1="15.24" y1="0" x2="15.24" y2="44.45" width="0.4064" layer="49"/>
 <text x="24.765" y="18.415" size="2.54" layer="25" font="vector" ratio="10" rot="R90">R</text>
 <text x="24.765" y="24.765" size="2.54" layer="25" font="vector" ratio="10" rot="R90">L</text>
@@
 <text x="6.35" y="26.035" size="1.778" layer="25" font="vector" ratio="20" rot="SR270">-</text>
 <text x="9.525" y="15.875" size="1.778" layer="25" font="vector" ratio="20" rot="R90">+</text>
+<wire x1="21.59" y1="22.225" x2="30.48" y2="22.225" width="0.4064" layer="25"/>
+<text x="13.97" y="40.64" size="1.778" layer="25" ratio="14" rot="SR0">RADIO</text>
 </plain>
 <attributes>
@@
 </autorouter>
 <elements>
-<element name="JP3" library="amp" package="1X02" value="OUT_R" x="26.035" y="13.335" smashed="yes" rot="R90">
-<attribute name="VALUE" x="29.21" y="10.795" size="1.27" layer="27" rot="R90"/>
-</element>
-<element name="JP2" library="amp" package="1X02" value="OUT_L" x="26.035" y="31.115" smashed="yes" rot="R270">
-<attribute name="VALUE" x="22.86" y="33.655" size="1.27" layer="27" rot="R270"/>
-</element>
+<element name="JP3" library="amp" package="1X02" value="OUT_R" x="26.035" y="13.335" smashed="yes" rot="R90"/>
+<element name="JP2" library="amp" package="1X02" value="OUT_L" x="26.035" y="31.115" smashed="yes" rot="R270"/>
 <element name="U$1" library="amp" package="3,0" value="" x="3.81" y="3.81" smashed="yes"/>
 <element name="U$2" library="amp" package="3,0" value="" x="3.81" y="40.64" smashed="yes"/>
@@
 <element name="U$4" library="amp" package="3,0" value="" x="26.67" y="3.81" smashed="yes"/>
 <element name="U1" library="amp" package="TEA5767" value="TEA5767" x="15.24" y="22.225" smashed="yes"/>
-<element name="IC1" library="amp" package="SOT223" value="LM1117S" x="15.24" y="8.89" smashed="yes" rot="R180">
-<attribute name="VALUE" x="17.78" y="10.2108" size="1.27" layer="27" rot="R180"/>
-</element>
+<element name="IC1" library="amp" package="SOT223" value="LM1117S" x="15.24" y="8.89" smashed="yes" rot="R180"/>
 <element name="JP1" library="amp" package="1X03" value="" x="4.445" y="27.94" smashed="yes" rot="R270">
 <attribute name="VALUE" x="1.27" y="31.75" size="1.27" layer="27" rot="R270"/>
@@
 <attribute name="VALUE" x="9.525" y="15.24" size="1.016" layer="27" ratio="10" rot="R90"/>
 </element>
-<element name="C1" library="amp" package="C0805K" value="10uF" x="10.16" y="8.89" smashed="yes" rot="R270">
-<attribute name="VALUE" x="8.26" y="9.89" size="1.016" layer="27" rot="R270"/>
-</element>
-<element name="C4" library="amp" package="C0805K" value="10uF" x="20.32" y="8.89" smashed="yes" rot="R270">
-<attribute name="VALUE" x="18.42" y="9.89" size="1.016" layer="27" rot="R270"/>
-</element>
-<element name="C2" library="amp" package="C0805K" value="1uF" x="26.035" y="25.4" smashed="yes" rot="R90">
-<attribute name="VALUE" x="27.935" y="24.4" size="1.016" layer="27" rot="R90"/>
-</element>
-<element name="C3" library="amp" package="C0805K" value="1uF" x="26.035" y="19.05" smashed="yes" rot="R270">
-<attribute name="VALUE" x="24.135" y="20.05" size="1.016" layer="27" rot="R270"/>
-</element>
+<element name="C1" library="amp" package="C0805K" value="10uF" x="10.16" y="8.89" smashed="yes" rot="R270"/>
+<element name="C4" library="amp" package="C0805K" value="10uF" x="20.32" y="8.89" smashed="yes" rot="R270"/>
+<element name="C2" library="amp" package="C0805K" value="1uF" x="26.035" y="25.4" smashed="yes" rot="R90"/>
+<element name="C3" library="amp" package="C0805K" value="1uF" x="26.035" y="19.05" smashed="yes" rot="R270"/>
+<element name="U$5" library="amp" package="FOX-1" value="" x="10.795" y="41.91"/>
 </elements>
 <signals>
@@
 </polygon>
 <via x="11.43" y="5.08" extent="1-16" drill="1" diameter="1.6764"/>
+<via x="11.43" y="2.54" extent="1-16" drill="1" diameter="1.6764"/>
+<via x="19.05" y="2.54" extent="1-16" drill="1" diameter="1.6764"/>
+<via x="19.05" y="5.08" extent="1-16" drill="1" diameter="1.6764"/>
 </signal>
 <signal name="SDA">
@@
 <wire x1="10.16" y1="9.89" x2="10.16" y2="12.04" width="0.4064" layer="1"/>
 </signal>
-<signal name="N$5">
-<via x="11.43" y="2.54" extent="1-16" drill="1" diameter="1.6764"/>
-</signal>
-<signal name="N$6">
-<via x="19.05" y="2.54" extent="1-16" drill="1" diameter="1.6764"/>
-</signal>
-<signal name="N$7">
-<via x="19.05" y="5.08" extent="1-16" drill="1" diameter="1.6764"/>
-</signal>
 </signals>
