File: pcb/PR038 - P27 (bass pre-amp)/P27_v3.brd (EAGLE design)
At the start: 41.9 x 64.8 mm, 52 parts, among them IC1 NE5532P, IC2 7815, IC3 7915, Q1 BC549

Commit message: 
Connections:
- net N$10 renamed TRB
- net N$13 renamed VOL
- net N$21 renamed OUT
- net N$25 renamed HI
- net N$26 renamed LOW
- net N$27 renamed IN
- net N$7 renamed MID
- net N$9 renamed BAS
Changed lines of the file:
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@@
 <wire x1="21.59" y1="52.07" x2="19.05" y2="52.07" width="0.4064" layer="16"/>
 </signal>
-<signal name="N$7">
+<signal name="MID">
 <contactref element="C6" pad="2"/>
 <contactref element="TRIMPOT" pad="4"/>
@@
 <wire x1="16.51" y1="59.69" x2="19.05" y2="57.15" width="0.4064" layer="16"/>
 </signal>
-<signal name="N$9">
+<signal name="BAS">
 <contactref element="C5" pad="2"/>
 <contactref element="TRIMPOT" pad="3"/>
@@
 <wire x1="19.05" y1="59.69" x2="21.59" y2="57.15" width="0.4064" layer="16"/>
 </signal>
-<signal name="N$10">
+<signal name="TRB">
 <contactref element="C4" pad="2"/>
 <contactref element="TRIMPOT" pad="2"/>
@@
 <wire x1="26.67" y1="52.07" x2="26.67" y2="48.26" width="0.4064" layer="16"/>
 </signal>
-<signal name="N$13">
+<signal name="VOL">
 <contactref element="TRIMPOT" pad="1"/>
 <contactref element="R8" pad="2"/>
@@
 <wire x1="30.48" y1="58.42" x2="29.21" y2="57.15" width="0.4064" layer="16"/>
 </signal>
-<signal name="N$21">
+<signal name="OUT">
 <contactref element="R12" pad="2"/>
 <contactref element="R13" pad="2"/>
@@
 <wire x1="35.56" y1="41.91" x2="36.83" y2="40.64" width="0.4064" layer="16"/>
 </signal>
-<signal name="N$27">
+<signal name="IN">
 <contactref element="MASTER" pad="1"/>
 <contactref element="C10" pad="1"/>
@@
 <wire x1="36.83" y1="7.62" x2="34.29" y2="5.08" width="0.4064" layer="16"/>
 </signal>
-<signal name="N$25">
+<signal name="HI">
 <contactref element="IN" pad="3"/>
 <contactref element="R1" pad="1"/>
 <wire x1="26.67" y1="5.08" x2="26.67" y2="8.89" width="0.4064" layer="16"/>
 </signal>
-<signal name="N$26">
+<signal name="LOW">
 <contactref element="IN" pad="2"/>
 <contactref element="R2" pad="1"/>
